File: TestOne/TestOne.kicad_pcb (KiCad board)
At the start: 2 copper layers, 28 parts, among them SW1 SW_Push, U1 ATmega32U4-AU, Y1 Crystal_GND24_Small

Commit message: Finished
Routing:
- net GND: track 138.0 -> 137.4 mm
- added copper zone on B.Cu, net GND
Other:
- board text added: "Keyboard Test One"
